File: kicad/spring-reverb/spring-reverb.kicad_sch (KiCad schematic)
At the start: 0 parts

Commit message: init kicad project
Parts:
- added C1, C2, C3: C, symbol Device:C
- added J1: Jack-DC, symbol Connector:Jack-DC
- added R1, R2, R3, R4: R, symbol Device:R
- added U1, U2: TL072, symbol Amplifier_Operational:TL072
Connections:
- new net: C3.1, U1.6 (-), U1.7
- new net: C2.1, U1.1, U1.2 (-)
- new net: R1.2, U1.3 (+), U1.5 (+)
- new net: R1.1, R2.2, R3.1, R4.1
- new net: C1.1, J1.2
- new net: R4.2, U2.3 (+)
- new net +9V: R2.1
- new net Earth: J1.1, R3.2

Commit message: Update KiCad schematic
Parts:
- removed C2, C3: C, symbol Device:C
- added C2, C3, C8: 100uF, symbol Device:C_Polarized
- added C4: 4,7nF, symbol Device:C
- added C5: 22nF, symbol Device:C
- added C6, C9: 100nF, symbol Device:C
- added C7: 47uF, symbol Device:C_Polarized
- added D1: 1N4007, Diode_THT:D_DO-41_SOD81_P10.16mm_Horizontal, symbol Diode:1N4007
- added J2: Jack-DC, symbol Connector:Jack-DC
- added R10: B100k, symbol Device:R_Potentiometer
- added R3: 1M, symbol Device:R
- added R4: 680 ohms, symbol Device:R
- added R5: B10k, symbol Device:R_Potentiometer
- added R6, R7: 47k, symbol Device:R
- added R8: 10k, symbol Device:R
- added R9: 6k8, symbol Device:R
- added SW1, SW2: ~, symbol Switch:SW_DPDT_x2
- C1: value C -> 100nF
- R1: value R -> 470k
- R11: renamed from R2; value R -> 470k
- R12: renamed from R3; value R -> 470k
- R2: renamed from R4; value R -> 470k
Connections:
- net +9V: now also C8.1, C9.2, D1.1 (K)
- net Earth: now also C7.2, C8.2, C9.1, D1.2 (A), J2.1, R10.3, R4.1, R9.2
- net at U1.6 (-), U1.7: now also C3.2
- net at U1.1, U1.2 (-): now also C2.2
- net at R1.2, U1.3 (+), U1.5 (+): now also C1.2
- net at R1.1, R11.2, R12.1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: now also C7.1
- net at R2.2, U2.3 (+): now also SW1.5 (B)
- net at U2.5 (+): now also R5.2, R6.1, R7.1
- net at U2.6 (-): now also R8.2, R9.1
- net at U2.7: now also C6.2, R8.1
- net at U2.1: now also R3.1, R5.1, R6.2, SW2.5 (B)
- net at U2.2 (-): now also R3.2, R4.2, SW2.2 (B)
- new net: C3.1, R5.3, R7.2
- new net: C4.2, SW2.1 (A)
- new net: C5.1, SW2.3 (C)
- new net: SW1.1 (A), SW1.4 (A)
- new net: C2.1, SW1.2 (B)
- new net: SW1.3 (C), SW1.6 (C)
- new net: C6.1, R10.1
- new net: J2.2, R10.2
- new net: C4.1, SW2.4 (A)
- new net: C5.2, SW2.6 (C)
Other:
- note added: "+4.5V"
- note added: "Accutronics 4BB3C1B"
- note added: "Accutronics 8BB2C1B"
- moved on the sheet: C1, R1, U1B, U2B

Commit message: rename potentiometers to RV1 and RV2
Parts:
- renumbered R12 to R10, R6 to R5, R7 to R6, R8 to R7, R9 to R8, R11 to R9, R5 to RV1, R10 to RV2
Changed lines of the file:
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@@
 		(dnp no)
 		(fields_autoplaced yes)
-		(property "Reference" "R9"
+		(property "Reference" "R8"
 			(at 212.09 143.5099 0)
 			(effects
@@
 			(project "spring-reverb"
 				(path "/4a6a507c-90a4-414f-880b-d22307af6194"
-					(reference "R9")
+					(reference "R8")
 					(unit 1)
 				)
@@
 		(dnp no)
 		(fields_autoplaced yes)
-		(property "Reference" "R7"
+		(property "Reference" "R6"
 			(at 195.58 142.24 90)
 			(effects
@@
 			(project "spring-reverb"
 				(path "/4a6a507c-90a4-414f-880b-d22307af6194"
-					(reference "R7")
+					(reference "R6")
 					(unit 1)
 				)
@@
 		(on_board yes)
 		(dnp no)
-		(property "Reference" "R11"
+		(property "Reference" "R9"
 			(at 58.674 34.29 0)
 			(effects
@@
 			(project ""
 				(path "/4a6a507c-90a4-414f-880b-d22307af6194"
-					(reference "R11")
+					(reference "R9")
 					(unit 1)
 				)
@@
 		(dnp no)
 		(fields_autoplaced yes)
-		(property "Reference" "R5"
+		(property "Reference" "RV1"
 			(at 186.69 120.6499 0)
 			(effects
@@
 			(project ""
 				(path "/4a6a507c-90a4-414f-880b-d22307af6194"
-					(reference "R5")
+					(reference "RV1")
 					(unit 1)
 				)
@@
 		(dnp no)
 		(fields_autoplaced yes)
-		(property "Reference" "R10"
+		(property "Reference" "RV2"
 			(at 245.11 128.27 90)
 			(effects
@@
 			(project "spring-reverb"
 				(path "/4a6a507c-90a4-414f-880b-d22307af6194"
-					(reference "R10")
+					(reference "RV2")
 					(unit 1)
 				)
@@
 		(on_board yes)
 		(dnp no)
-		(property "Reference" "R12"
+		(property "Reference" "R10"
 			(at 58.674 46.482 0)
 			(effects
@@
 			(project ""
 				(path "/4a6a507c-90a4-414f-880b-d22307af6194"
-					(reference "R12")
+					(reference "R10")
 					(unit 1)
 				)
@@
 		(dnp no)
 		(fields_autoplaced yes)
-		(property "Reference" "R6"
+		(property "Reference" "R5"
 			(at 195.58 91.44 90)
 			(effects
@@
 			(project "spring-reverb"
 				(path "/4a6a507c-90a4-414f-880b-d22307af6194"
-					(reference "R6")
+					(reference "R5")
 					(unit 1)
 				)
@@
 		(dnp no)
 		(fields_autoplaced yes)
-		(property "Reference" "R8"
+		(property "Reference" "R7"
 			(at 218.44 130.81 90)
 			(effects
@@
 			(project "spring-reverb"
 				(path "/4a6a507c-90a4-414f-880b-d22307af6194"
-					(reference "R8")
-					(unit 1)
-				)
+					(reference "R7")
+					(unit 1)
+				)
